File: USB_HUB_ADAPTER/USB_HUB_ADAPTER.kicad_sch (KiCad schematic)
At the start: 59 parts, among them IC1 TUSB564, J1 SD-106M, J2 TF-115-BCP9, J3 TYPEC-324DBW-ACP24A, J4 USB3_A, J5 USB3_A, U1 SY6280, U2 SY6280

Commit message: v2 layout update
Parts:
- removed TP1: VBUS_TP, brilliant-kicad-library:TestPoint_Pad_D0.9mm, symbol Connector:TestPoint
- added TP_vbus1: VBUS_TP, brilliant-kicad-library:TestPoint_Pad_D0.9mm, symbol Connector:TestPoint
Connections:
- net SYS_PWR: now also TP_vbus1.1
- net USB3DN_4_D_N: now also D7.2 (IO1), J5.2 (D-); no longer D4.2 (IO1), J3.A7 (D-), J3.B7 (D-)
- net USB3DN_4_D_P: now also D7.3 (IO2), J5.3 (D+); no longer D4.3 (IO2), J3.A6 (D+), J3.B6 (D+)
- net USB3DN_5_D_N: now also D4.2 (IO1), J3.A7 (D-), J3.B7 (D-); no longer D7.2 (IO1), J5.2 (D-)
- net USB3DN_5_D_P: now also D4.3 (IO2), J3.A6 (D+), J3.B6 (D+); no longer D7.3 (IO2), J5.3 (D+)
- net USB3DN_RXD_4_N: now also D9.2 (IO1), J5.5 (SSRX-); no longer D6.2 (IO1), J3.B10 (RX1-)
- net USB3DN_RXD_4_P: now also D9.3 (IO2), J5.6 (SSRX+); no longer D6.3 (IO2), J3.B11 (RX1+)
- net USB3DN_RXD_5_N: now also D6.2 (IO1), J3.B10 (RX1-); no longer D9.2 (IO1), J5.5 (SSRX-)
- net USB3DN_RXD_5_P: now also D6.3 (IO2), J3.B11 (RX1+); no longer D9.3 (IO2), J5.6 (SSRX+)
- net USB3DN_TXD_4_N: now also D8.2 (IO1), J5.8 (SSTX-); no longer D5.2 (IO1), J3.A3 (TX1-)
- net USB3DN_TXD_4_P: now also D8.3 (IO2), J5.9 (SSTX+); no longer D5.3 (IO2), J3.A2 (TX1+)
- net USB3DN_TXD_5_N: now also D5.2 (IO1), J3.A3 (TX1-); no longer D8.2 (IO1), J5.8 (SSTX-)
- net USB3DN_TXD_5_P: now also D5.3 (IO2), J3.A2 (TX1+); no longer D8.3 (IO2), J5.9 (SSTX+)

Commit message: completed routing and layout
Connections:
- no-connect marks 17 -> 19
Changed lines of the file:
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@@
   (no_connect (at 526.415 193.675))
   (no_connect (at 526.415 201.295))
+  (no_connect (at 270.51 398.145))
+  (no_connect (at 270.51 317.5))
   (no_connect (at 339.09 237.49))
   (no_connect (at 339.09 230.505))
@@
     (stroke (width 0) (type default) (color 0 0 0 0))
   )
-  (wire (pts (xy 270.51 317.5) (xy 270.51 398.145))
-    (stroke (width 0) (type default) (color 0 0 0 0))
-  )
   (wire (pts (xy 497.205 40.64) (xy 511.81 40.64))
     (stroke (width 0) (type default) (color 0 0 0 0))
@@
       (reference "#PWR0172") (unit 1) (value "GND") (footprint "")
     )
+    (path "/5e9cc844-d5be-46c7-81dd-e2c0bb534986/9d1626b8-ddd2-4ba3-8811-595dd6deef9b"
+      (reference "#PWR0173") (unit 1) (value "+3V3") (footprint "")
+    )
+    (path "/5e9cc844-d5be-46c7-81dd-e2c0bb534986/e5d74059-9bc6-4ed7-9c48-b19642d11fee"
+      (reference "#PWR0174") (unit 1) (value "GND") (footprint "")
+    )
+    (path "/5e9cc844-d5be-46c7-81dd-e2c0bb534986/58ead586-7fd3-4b93-8691-4969eef780c4"
+      (reference "#PWR0175") (unit 1) (value "+1V8") (footprint "")
+    )
     (path "/5b0d2f65-a75c-4dcc-89e9-1112dd9dab29"
       (reference "C1") (unit 1) (value "100n") (footprint "Capacitor_SMD:C_0805_2012Metric")
@@
       (reference "C101") (unit 1) (value "22p") (footprint "Capacitor_SMD:C_0805_2012Metric")
     )
+    (path "/5e9cc844-d5be-46c7-81dd-e2c0bb534986/0ac3ea24-362e-4170-b944-13398f9ec521"
+      (reference "C102") (unit 1) (value "1u") (footprint "Capacitor_SMD:C_0402_1005Metric")
+    )
     (path "/51546a8a-1c7b-4f62-9a88-06894d757d3a/00000000-0000-0000-0000-000061de3b39"
       (reference "C103") (unit 1) (value "1uF_50V") (footprint "Capacitor_SMD:C_0402_1005Metric")
@@
       (reference "C137") (unit 1) (value "10uF_1mOHM_402") (footprint "Capacitor_SMD:C_0402_1005Metric")
     )
+    (path "/5e9cc844-d5be-46c7-81dd-e2c0bb534986/d9616a13-0e9b-45fa-a4da-e855757b7c43"
+      (reference "C138") (unit 1) (value "1u") (footprint "Capacitor_SMD:C_0402_1005Metric")
+    )
     (path "/104488d6-e960-4cda-b8ea-7eeb7abacfe4"
       (reference "CC1") (unit 1) (value "CC1") (footprint "greencharge-footprints:TP_PAD_1.5x0.8")
@@
       (reference "U12") (unit 1) (value "TLV320AIC3104IRHBR") (footprint "Package_DFN_QFN:VQFN-32-1EP_5x5mm_P0.5mm_EP3.5x3.5mm")
     )
+    (path "/5e9cc844-d5be-46c7-81dd-e2c0bb534986/c7d1fd41-699d-47e6-a842-863e032220f9"
+      (reference "U13") (unit 1) (value "AP2127N-1.8") (footprint "Package_TO_SOT_SMD:SOT-23")
+    )
     (path "/2663f88e-7e76-4227-8baf-f7576dcda145"
