File: USB_HUB_ADAPTER/audio_codec_TLV320AIC3104IRHBR.kicad_sch (KiCad schematic)
At the start: 17 parts, among them J7 PL320E, U12 TLV320AIC3104IRHBR

Commit message: v2 layout update
Parts:
- C72, C73, C74, C75, C76, C77, C78, C79, C80, C94: footprint (none) -> Capacitor_SMD:C_0402_1005Metric
- J7: value PL320E -> 54-00178; footprint Connector_Audio:Jack_3.5mm_PJ320E_Horizontal -> Connector_Audio:Jack_3.5mm_PJ311_Horizontal
Connections:
- net +3V3: now also U12.31 (~{RESET})
- net GND: now also J7.2 (G); no longer J7.G
- net at C96.2: now also J7.4 (t); no longer J7.T
- net at C95.2: now also J7.3 (s); no longer J7.S
- no-connect marks 3 -> 12
Changed lines of the file:
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@@
   (junction (at 167.64 36.83) (diameter 0) (color 0 0 0 0)
   )
+  (no_connect (at 165.1 90.17))
+  (no_connect (at 113.03 90.17))
+  (no_connect (at 113.03 92.71))
+  (no_connect (at 113.03 95.25))
+  (no_connect (at 113.03 97.79))
+  (no_connect (at 113.03 100.33))
+  (no_connect (at 113.03 102.87))
+  (no_connect (at 165.1 64.77))
+  (no_connect (at 165.1 67.31))
   (no_connect (at 165.1 92.71))
   (no_connect (at 165.1 78.74))
@@
     (stroke (width 0) (type default) (color 0 0 0 0))
   )
+  (wire (pts (xy 105.41 54.61) (xy 113.03 54.61))
+    (stroke (width 0) (type default) (color 0 0 0 0))
+  )
   (wire (pts (xy 60.325 60.96) (xy 60.325 59.69))
     (stroke (width 0) (type default) (color 0 0 0 0))
@@
   )
   (wire (pts (xy 139.7 38.1) (xy 139.7 44.45))
+    (stroke (width 0) (type default) (color 0 0 0 0))
+  )
+  (wire (pts (xy 105.41 53.34) (xy 105.41 54.61))
     (stroke (width 0) (type default) (color 0 0 0 0))
   )
@@
     (effects (font (size 1.27 1.27)) (justify right))
   )
+  (symbol (lib_id "power:+3V3") (at 105.41 53.34 0) (unit 1)
+    (in_bom yes) (on_board yes) (fields_autoplaced)
+    (property "Reference" "#PWR0147" (id 0) (at 105.41 57.15 0)
+      (effects (font (size 1.27 1.27)) hide)
+    )
+    (property "Value" "+3V3" (id 1) (at 105.41 48.26 0))
+    (property "Footprint" "" (id 2) (at 105.41 53.34 0)
+      (effects (font (size 1.27 1.27)) hide)
+    )
+    (property "Datasheet" "" (id 3) (at 105.41 53.34 0)
+      (effects (font (size 1.27 1.27)) hide)
+    )
+    (pin "1")
+  )
   (symbol (lib_id "Device:R_US") (at 60.325 64.77 0) (unit 1)
     (in_bom yes) (on_board yes)
@@
       (effects (font (size 1.27 1.27)) (justify left))
     )
-    (property "Footprint" "" (id 2) (at 181.61 40.64 0)
+    (property "Footprint" "Capacitor_SMD:C_0402_1005Metric" (id 2) (at 181.61 40.64 0)
       (effects (font (size 1.27 1.27)) hide)
     )
@@
       (effects (font (size 1.27 1.27)) (justify left))
     )
-    (property "Footprint" "" (id 2) (at 111.76 40.64 0)
+    (property "Footprint" "Capacitor_SMD:C_0402_1005Metric" (id 2) (at 111.76 40.64 0)
       (effects (font (size 1.27 1.27)) hide)
     )
@@
   (symbol (lib_id "Connector:AudioJack2_Ground") (at 217.17 53.975 0) (mirror y) (unit 1)
     (in_bom yes) (on_board yes)
-    (property "Reference" "J7" (id 0) (at 216.3572 45.72 0))
-    (property "Value" "PL320E" (id 1) (at 216.3572 48.0314 0))
-    (property "Footprint" "Connector_Audio:Jack_3.5mm_PJ320E_Horizontal" (id 2) (at 217.17 53.975 0)
+    (property "Reference" "J7" (id 0) (at 217.9828 45.72 0))
+    (property "Value" "54-00178" (id 1) (at 217.9828 48.0314 0))
+    (property "Footprint" "Connector_Audio:Jack_3.5mm_PJ311_Horizontal" (id 2) (at 217.17 53.975 0)
       (effects (font (size 1.27 1.27)) hide)
     )
@@
       (effects (font (size 1.27 1.27)) hide)
     )
-    (pin "G")
-    (pin "S")
-    (pin "T")
+    (pin "2")
+    (pin "3")
+    (pin "4")
   )
   (symbol (lib_id "Device:C_Small") (at 143.51 40.64 0) (unit 1)
@@
       (effects (font (size 1.27 1.27)) (justify left))
     )
-    (property "Footprint" "" (id 2) (at 143.51 40.64 0)
+    (property "Footprint" "Capacitor_SMD:C_0402_1005Metric" (id 2) (at 143.51 40.64 0)
       (effects (font (size 1.27 1.27)) hide)
     )
@@
       (effects (font (size 1.27 1.27)) (justify left))
     )
-    (property "Footprint" "" (id 2) (at 115.57 24.13 0)
+    (property "Footprint" "Capacitor_SMD:C_0402_1005Metric" (id 2) (at 115.57 24.13 0)
       (effects (font (size 1.27 1.27)) hide)
     )
@@
       (effects (font (size 1.27 1.27)) (justify left))
     )
-    (property "Footprint" "" (id 2) (at 151.13 33.02 0)
+    (property "Footprint" "Capacitor_SMD:C_0402_1005Metric" (id 2) (at 151.13 33.02 0)
       (effects (font (size 1.27 1.27)) hide)
     )
@@
       (effects (font (size 1.27 1.27)) (justify left))
     )
-    (property "Footprint" "" (id 2) (at 151.13 40.64 0)
+    (property "Footprint" "Capacitor_SMD:C_0402_1005Metric" (id 2) (at 151.13 40.64 0)
       (effects (font (size 1.27 1.27)) hide)
     )
@@
       (effects (font (size 1.27 1.27)) (justify left))
     )
-    (property "Footprint" "" (id 2) (at 120.65 40.64 0)
+    (property "Footprint" "Capacitor_SMD:C_0402_1005Metric" (id 2) (at 120.65 40.64 0)
       (effects (font (size 1.27 1.27)) hide)
     )
@@
       (effects (font (size 1.27 1.27)) (justify left))
     )
-    (property "Footprint" "" (id 2) (at 142.24 33.02 0)
+    (property "Footprint" "Capacitor_SMD:C_0402_1005Metric" (id 2) (at 142.24 33.02 0)
       (effects (font (size 1.27 1.27)) hide)
     )
@@
       (effects (font (size 1.27 1.27)) (justify left))
     )
-    (property "Footprint" "" (id 2) (at 172.72 40.64 0)
+    (property "Footprint" "Capacitor_SMD:C_0402_1005Metric" (id 2) (at 172.72 40.64 0)
       (effects (font (size 1.27 1.27)) hide)
     )
@@
       (effects (font (size 1.27 1.27)) (justify left))
     )
-    (property "Footprint" "" (id 2) (at 124.46 24.13 0)
-      (effects (font (size 1.27 1.27)) hide)
-    )
+    (property "Footprint" "Capacitor_SMD:C_0402_1005Metric" (id 2) (at 124.46 24.13 0)
+      (effects (font (size 1.27 1.27)) hide)
+    )

Commit message: completed routing and layout
Parts:
- added C102, C138: 1u, Capacitor_SMD:C_0402_1005Metric, symbol Device:C_Small
- added U13: AP2127N-1.8, Package_TO_SOT_SMD:SOT-23, symbol Regulator_Linear:AP2127N-1.8
Connections:
- net +1V8: now also C138.1, U13.2 (VO)
- net +3V3: now also C102.1, U13.3 (VI)
- net GND: now also C102.2, C138.2, U13.1 (GND)
Changed lines of the file:
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@@
 (kicad_sch (version 20211123) (generator eeschema)
   (paper "A4")
+  (junction (at 235.585 20.955) (diameter 0) (color 0 0 0 0)
+  )
   (junction (at 139.7 115.57) (diameter 0) (color 0 0 0 0)
   )
@@
   )
   (junction (at 139.7 30.48) (diameter 0) (color 0 0 0 0)
+  )
+  (junction (at 207.01 20.955) (diameter 0) (color 0 0 0 0)
+  )
+  (junction (at 222.25 33.02) (diameter 0) (color 0 0 0 0)
   )
   (junction (at 142.24 115.57) (diameter 0) (color 0 0 0 0)
@@
     (stroke (width 0) (type default) (color 0 0 0 0))
   )
+  (wire (pts (xy 207.01 19.685) (xy 207.01 20.955))
+    (stroke (width 0) (type default) (color 0 0 0 0))
+  )
   (wire (pts (xy 151.13 35.56) (xy 158.75 35.56))
     (stroke (width 0) (type default) (color 0 0 0 0))
@@
     (stroke (width 0) (type default) (color 0 0 0 0))
   )
+  (wire (pts (xy 235.585 20.955) (xy 229.87 20.955))
+    (stroke (width 0) (type default) (color 0 0 0 0))
+  )
   (wire (pts (xy 137.16 111.76) (xy 137.16 115.57))
     (stroke (width 0) (type default) (color 0 0 0 0))
@@
     (stroke (width 0) (type default) (color 0 0 0 0))
   )
+  (wire (pts (xy 235.585 33.02) (xy 235.585 27.94))
+    (stroke (width 0) (type default) (color 0 0 0 0))
+  )
   (wire (pts (xy 134.62 111.76) (xy 134.62 115.57))
     (stroke (width 0) (type default) (color 0 0 0 0))
   )
+  (wire (pts (xy 207.01 27.94) (xy 207.01 33.02))
+    (stroke (width 0) (type default) (color 0 0 0 0))
+  )
   (wire (pts (xy 120.65 36.83) (xy 111.76 36.83))
     (stroke (width 0) (type default) (color 0 0 0 0))
@@
     (stroke (width 0) (type default) (color 0 0 0 0))
   )
+  (wire (pts (xy 222.25 33.02) (xy 235.585 33.02))
+    (stroke (width 0) (type default) (color 0 0 0 0))
+  )
   (wire (pts (xy 165.1 60.96) (xy 194.31 60.96))
     (stroke (width 0) (type default) (color 0 0 0 0))
@@
     (stroke (width 0) (type default) (color 0 0 0 0))
   )
+  (wire (pts (xy 222.25 28.575) (xy 222.25 33.02))
+    (stroke (width 0) (type default) (color 0 0 0 0))
+  )
   (wire (pts (xy 111.76 43.18) (xy 111.76 44.45))
     (stroke (width 0) (type default) (color 0 0 0 0))
@@
     (stroke (width 0) (type default) (color 0 0 0 0))
   )
+  (wire (pts (xy 207.01 20.955) (xy 214.63 20.955))
+    (stroke (width 0) (type default) (color 0 0 0 0))
+  )
   (wire (pts (xy 143.51 38.1) (xy 151.13 38.1))
     (stroke (width 0) (type default) (color 0 0 0 0))
@@
     (stroke (width 0) (type default) (color 0 0 0 0))
   )
+  (wire (pts (xy 207.01 33.02) (xy 222.25 33.02))
+    (stroke (width 0) (type default) (color 0 0 0 0))
+  )
   (wire (pts (xy 139.7 38.1) (xy 143.51 38.1))
     (stroke (width 0) (type default) (color 0 0 0 0))
@@
     (stroke (width 0) (type default) (color 0 0 0 0))
   )
+  (wire (pts (xy 235.585 22.86) (xy 235.585 20.955))
+    (stroke (width 0) (type default) (color 0 0 0 0))
+  )
   (wire (pts (xy 142.24 115.57) (xy 144.78 115.57))
+    (stroke (width 0) (type default) (color 0 0 0 0))
+  )
+  (wire (pts (xy 207.01 20.955) (xy 207.01 22.86))
     (stroke (width 0) (type default) (color 0 0 0 0))
   )
@@
     (pin "1")
   )
+  (symbol (lib_id "Device:C_Small") (at 207.01 25.4 0) (unit 1)
+    (in_bom yes) (on_board yes) (fields_autoplaced)
+    (property "Reference" "C102" (id 0) (at 209.55 24.1362 0)
+      (effects (font (size 1.27 1.27)) (justify left))
+    )
+    (property "Value" "1u" (id 1) (at 209.55 26.6762 0)
+      (effects (font (size 1.27 1.27)) (justify left))
+    )
+    (property "Footprint" "Capacitor_SMD:C_0402_1005Metric" (id 2) (at 207.01 25.4 0)
+      (effects (font (size 1.27 1.27)) hide)
+    )
+    (property "Datasheet" "~" (id 3) (at 207.01 25.4 0)
+      (effects (font (size 1.27 1.27)) hide)
+    )
+    (pin "1")
+    (pin "2")
+  )
   (symbol (lib_id "Device:R_US") (at 60.325 64.77 0) (unit 1)
     (in_bom yes) (on_board yes)
@@
     (pin "1")
   )
+  (symbol (lib_id "power:+1V8") (at 235.585 20.955 0) (unit 1)
+    (in_bom yes) (on_board yes) (fields_autoplaced)
+    (property "Reference" "#PWR0175" (id 0) (at 235.585 24.765 0)
+      (effects (font (size 1.27 1.27)) hide)
+    )
+    (property "Value" "+1V8" (id 1) (at 235.585 15.875 0))
+    (property "Footprint" "" (id 2) (at 235.585 20.955 0)
+      (effects (font (size 1.27 1.27)) hide)
+    )
+    (property "Datasheet" "" (id 3) (at 235.585 20.955 0)
+      (effects (font (size 1.27 1.27)) hide)
+    )
+    (pin "1")
+  )
   (symbol (lib_id "power:GND") (at 217.17 60.96 0) (unit 1)
     (in_bom yes) (on_board yes)
@@
     (pin "1")
     (pin "2")
+  )
+  (symbol (lib_id "power:+3V3") (at 207.01 19.685 0) (unit 1)
+    (in_bom yes) (on_board yes) (fields_autoplaced)
+    (property "Reference" "#PWR0173" (id 0) (at 207.01 23.495 0)
+      (effects (font (size 1.27 1.27)) hide)
+    )
+    (property "Value" "+3V3" (id 1) (at 207.01 14.605 0))
+    (property "Footprint" "" (id 2) (at 207.01 19.685 0)
+      (effects (font (size 1.27 1.27)) hide)
+    )
+    (property "Datasheet" "" (id 3) (at 207.01 19.685 0)
+      (effects (font (size 1.27 1.27)) hide)
+    )
+    (pin "1")
   )
   (symbol (lib_id "power:GND") (at 115.57 27.94 0) (unit 1)
@@
     (pin "1")
   )
+  (symbol (lib_id "Regulator_Linear:AP2127N-1.8") (at 222.25 20.955 0) (unit 1)
+    (in_bom yes) (on_board yes) (fields_autoplaced)
+    (property "Reference" "U13" (id 0) (at 222.25 13.97 0))
+    (property "Value" "AP2127N-1.8" (id 1) (at 222.25 16.51 0))
+    (property "Footprint" "Package_TO_SOT_SMD:SOT-23" (id 2) (at 222.25 15.24 0)
+      (effects (font (size 1.27 1.27) italic) hide)
+    )
+    (property "Datasheet" "https://www.diodes.com/assets/Datasheets/AP2127.pdf" (id 3) (at 222.25 20.955 0)
+      (effects (font (size 1.27 1.27)) hide)
+    )
+    (pin "1")
+    (pin "2")
+    (pin "3")
+  )
   (symbol (lib_id "Device:C_Small") (at 124.46 24.13 0) (unit 1)
     (in_bom yes) (on_board yes) (fields_autoplaced)
@@
     (pin "2")
   )
+  (symbol (lib_id "Device:C_Small") (at 235.585 25.4 0) (unit 1)
+    (in_bom yes) (on_board yes) (fields_autoplaced)
+    (property "Reference" "C138" (id 0) (at 238.125 24.1362 0)
+      (effects (font (size 1.27 1.27)) (justify left))
+    )
+    (property "Value" "1u" (id 1) (at 238.125 26.6762 0)
+      (effects (font (size 1.27 1.27)) (justify left))
+    )
+    (property "Footprint" "Capacitor_SMD:C_0402_1005Metric" (id 2) (at 235.585 25.4 0)
+      (effects (font (size 1.27 1.27)) hide)
+    )
+    (property "Datasheet" "~" (id 3) (at 235.585 25.4 0)
+      (effects (font (size 1.27 1.27)) hide)
+    )
+    (pin "1")
+    (pin "2")
+  )
+  (symbol (lib_id "power:GND") (at 222.25 33.02 0) (unit 1)
+    (in_bom yes) (on_board yes)
+    (property "Reference" "#PWR0174" (id 0) (at 222.25 39.37 0)
+      (effects (font (size 1.27 1.27)) hide)
+    )
+    (property "Value" "GND" (id 1) (at 222.25 36.83 0))
+    (property "Footprint" "" (id 2) (at 222.25 33.02 0)
+      (effects (font (size 1.27 1.27)) hide)
+    )
+    (property "Datasheet" "" (id 3) (at 222.25 33.02 0)
+      (effects (font (size 1.27 1.27)) hide)
+    )
+    (pin "1")
+  )
   (symbol (lib_id "Device:R_US") (at 67.31 64.77 0) (unit 1)
